File: dram-cart.sch (KiCad schematic (older format))
At the start: 7 parts, among them CON1 Conn_02x20_Odd_Even, U1 W25Q128JVSIQ, U2 IS42S16400J-xC

Commit message: Rev.B of Schematic and PCB
This corrects errors in Rev.A where the wrong pins were used for some DQ signals.

Signed-off-by: Jacob Creedon <jcreedon@gmail.com>
Parts:
- removed C3, C4: 100n, Capacitor_SMD:C_0603_1608Metric, symbol Device:C_Small
- removed U2: IS42S16400J-xC, IS42S16400J-6TL:SOP80P1176X120-54N, symbol Memory_RAM:IS42S16400J-xC
- added U2: TSOP-II-54-x8, Package_SO:TSOP-II-54_22.2x10.16mm_P0.8mm, symbol ram:TSOP-II-54-x8
Connections:
- wire segments 40 -> 36
Other:
- note removed: "Notes:\n- U1 can be any serial flash chip compatible with the Lattice ECP5 FPGA \n series. Something with 4MiB >= size >= 16MiB is preferred.\n- Max power draw from 3V3: 500mA\n- Max power draw from 5V: 300mA\n- Max draw from Vbat: whatever the batteries can supply\n- Note that 5V is generated by a boost converter from the battery \n voltage, it is NOT the 5V USB line.\n- CON1 connects to the bad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"
- moved on the sheet: C1, C2, CON1, U1
